File: DeskLight.brd (EAGLE design)
At the start: 44.5 x 58.4 mm, 39 parts, among them IC1 REG1117, T1 MMBT2222, T2 MMBT2222, T3 MJD122, T4 MJD122, T5 MJD122, U1 ESP32-WROOM-32D, U2 CH340C

Commit message: added comp. values
Parts:
- J1: value (none) -> Würth Elektronik SD Connector 693071020811
- R1, R2, R3: value (none) -> 10k
Changed lines of the file:
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@@
 <drawing>
 <settings>
-<setting alwaysvectorfont="no"/>
+<setting alwaysvectorfont="yes"/>
 <setting verticaltext="up"/>
 </settings>
@@
 <attribute name="VALUE" x="19.812" y="11.176" size="1.016" layer="27" font="vector" ratio="15" rot="R90"/>
 </element>
-<element name="J1" library="693071030811_Eagle_WR-CRD_rev20b" package="693071020811" package3d_urn="urn:adsk.eagle:package:16444883/2" value="" x="32.0675" y="54.2925" smashed="yes" rot="R180">
+<element name="J1" library="693071030811_Eagle_WR-CRD_rev20b" package="693071020811" package3d_urn="urn:adsk.eagle:package:16444883/2" value="Würth Elektronik SD Connector 693071020811" x="32.0675" y="54.2925" smashed="yes" rot="R180">
 <attribute name="DATASHEET-URL" value="https://www.we-online.com/catalog/datasheet/693071020811.pdf" x="-4.7625" y="91.1225" size="1.778" layer="27" rot="R180" display="off"/>
 <attribute name="GERDER" value="Socket" x="-4.7625" y="91.1225" size="1.778" layer="27" rot="R180" display="off"/>
@@
 <attribute name="PINS" value=" 8 " x="-4.7625" y="91.1225" size="1.778" layer="27" rot="R180" display="off"/>
 <attribute name="TYPE" value="Push &amp; Push" x="-4.7625" y="91.1225" size="1.778" layer="27" rot="R180" display="off"/>
-<attribute name="VALUE" x="22.6675" y="46.8925" size="1.27" layer="27" rot="R180"/>
 </element>
 <element name="RX" library="led" library_urn="urn:adsk.eagle:library:259" package="CHIP-LED0603" package3d_urn="urn:adsk.eagle:package:15819/3" value="BLUE" x="38.1" y="5.3975" smashed="yes">
@@
 <attribute name="VALUE" x="31.85" y="57.41" size="1.016" layer="28" font="vector" ratio="15" rot="MR0"/>
 </element>
-<element name="R1" library="rcl" library_urn="urn:adsk.eagle:library:334" package="R0603" package3d_urn="urn:adsk.eagle:package:23555/3" value="" x="23.1775" y="27.6225" smashed="yes" rot="R90">
+<element name="R1" library="rcl" library_urn="urn:adsk.eagle:library:334" package="R0603" package3d_urn="urn:adsk.eagle:package:23555/3" value="10k" x="23.1775" y="27.6225" smashed="yes" rot="R90">
 <attribute name="NAME" x="21.9075" y="26.9875" size="1.016" layer="25" font="vector" ratio="15" rot="R90"/>
 <attribute name="POPULARITY" value="77" x="95.5675" y="74.6125" size="1.778" layer="27" rot="R90" display="off"/>
@@
 <attribute name="VALUE" x="19.05" y="28.575" size="1.016" layer="27" font="vector" ratio="15" rot="R90"/>
 </element>
-<element name="R2" library="rcl" library_urn="urn:adsk.eagle:library:334" package="R0603" package3d_urn="urn:adsk.eagle:package:23555/3" value="" x="30.1625" y="27.6225" smashed="yes" rot="R90">
+<element name="R2" library="rcl" library_urn="urn:adsk.eagle:library:334" package="R0603" package3d_urn="urn:adsk.eagle:package:23555/3" value="10k" x="30.1625" y="27.6225" smashed="yes" rot="R90">
 <attribute name="NAME" x="28.8925" y="26.67" size="1.016" layer="25" font="vector" ratio="15" rot="R90"/>
 <attribute name="POPULARITY" value="77" x="102.5525" y="78.4225" size="1.778" layer="27" rot="R90" display="off"/>
@@
 <attribute name="VALUE" x="32.0675" y="26.9875" size="1.27" layer="27" rot="R90"/>
 </element>
-<element name="R3" library="rcl" library_urn="urn:adsk.eagle:library:334" package="R0603" package3d_urn="urn:adsk.eagle:package:23555/3" value="" x="37.1475" y="27.6225" smashed="yes" rot="R90">
+<element name="R3" library="rcl" library_urn="urn:adsk.eagle:library:334" package="R0603" package3d_urn="urn:adsk.eagle:package:23555/3" value="10k" x="37.1475" y="27.6225" smashed="yes" rot="R90">
 <attribute name="NAME" x="35.8775" y="26.67" size="1.016" layer="25" font="vector" ratio="15" rot="R90"/>
 <attribute name="POPULARITY" value="77" x="109.5375" y="82.2325" size="1.778" layer="27" rot="R90" display="off"/>
