File: DeskLight.sch (EAGLE design)
At the start: 39 parts, among them IC1 REG1117, T1 MMBT2222, T2 MMBT2222, T3 MJD122, T4 MJD122, T5 MJD122, U1 ESP32-WROOM-32D, U2 CH340C

Commit message: added comp. values
Parts:
- J1: value (none) -> Würth Elektronik SD Connector 693071020811
- R1, R2, R3: value (none) -> 10k
Changed lines of the file:
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@@
 </classes>
 <parts>
-<part name="J1" library="693071030811_Eagle_WR-CRD_rev20b" deviceset="693071020811" device="" package3d_urn="urn:adsk.eagle:package:16444883/2"/>
+<part name="J1" library="693071030811_Eagle_WR-CRD_rev20b" deviceset="693071020811" device="" package3d_urn="urn:adsk.eagle:package:16444883/2" value="Würth Elektronik SD Connector 693071020811"/>
 <part name="IC1" library="burr-brown" library_urn="urn:adsk.eagle:library:111" deviceset="REG1117" device="" package3d_urn="urn:adsk.eagle:package:4940/1"/>
 <part name="C1" library="rcl" library_urn="urn:adsk.eagle:library:334" deviceset="CPOL-EU" device="CT3216" package3d_urn="urn:adsk.eagle:package:23327/2" value="22uF"/>
 <part name="GND1" library="supply1" library_urn="urn:adsk.eagle:library:371" deviceset="GND" device=""/>
-<part name="R1" library="rcl" library_urn="urn:adsk.eagle:library:334" deviceset="R-US_" device="R0603" package3d_urn="urn:adsk.eagle:package:23555/3"/>
-<part name="R2" library="rcl" library_urn="urn:adsk.eagle:library:334" deviceset="R-US_" device="R0603" package3d_urn="urn:adsk.eagle:package:23555/3"/>
-<part name="R3" library="rcl" library_urn="urn:adsk.eagle:library:334" deviceset="R-US_" device="R0603" package3d_urn="urn:adsk.eagle:package:23555/3"/>
+<part name="R1" library="rcl" library_urn="urn:adsk.eagle:library:334" deviceset="R-US_" device="R0603" package3d_urn="urn:adsk.eagle:package:23555/3" value="10k"/>
+<part name="R2" library="rcl" library_urn="urn:adsk.eagle:library:334" deviceset="R-US_" device="R0603" package3d_urn="urn:adsk.eagle:package:23555/3" value="10k"/>
+<part name="R3" library="rcl" library_urn="urn:adsk.eagle:library:334" deviceset="R-US_" device="R0603" package3d_urn="urn:adsk.eagle:package:23555/3" value="10k"/>
 <part name="GND2" library="supply1" library_urn="urn:adsk.eagle:library:371" deviceset="GND" device=""/>
 <part name="U1" library="ESP32-WROOM-32D" deviceset="ESP32-WROOM-32D" device=""/>
